File: rocket2-adapter-board-universal.kicad_sch (KiCad schematic)
At the start: 6 parts, among them J1 DE15_Socket_HighDensity_Mount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

Commit message: BOM Generation Available + Standard KiCad Library
Added webpages for JLCPCB pre-assembly BOM. Added new standardized KiCAD library.
Parts:
- removed GX-16: J1, UCIRP-KiCAD-Lib:GX16-4, symbol UCIRP-KiCAD-Lib:GX16
- added J2: Conn_01x03_Socket, symbol Connector:Conn_01x03_Socket
- added J3: Conn_01x02_Socket, UCIRP-KiCAD-Lib:Solenoid TH, symbol Connector:Conn_01x02_Socket
- added J4: Conn_01x04_Socket, UCIRP-KiCAD-Lib:Load Cell Port, symbol Connector:Conn_01x04_Socket
- added VR1: R_Potentiometer, symbol Device:R_Potentiometer
- D1: value 5.5V -> ~27V
- R1: value 0/1k -> 0
Connections:
- net AIN+: now also J4.4 (Pin_4)
- net AIN-: now also J4.1 (Pin_1)
- net GND: now also J2.3 (Pin_3), J3.2 (Pin_2), J4.3 (Pin_3), VR1.1
- net VBUS: now also J2.1 (Pin_1), J3.1 (Pin_1), VR1.3
- net VIN: now also J4.2 (Pin_2)
- new net VOUT: VR1.2
- new net V_SIGNAL: J2.2 (Pin_2)
Other:
- note added: "LOAD CELL PORT"
- note added: "POTENTIOMETER PORT"
- note added: "PRESSURE TRANSDUCER PORT"
- note added: "SOLENOID PORT"
- note removed: "GX16 CONNECTOR"
- moved on the sheet: D1, F1, J1, R1, R2
