File: rocket2-adapter-board-universal.kicad_sch (KiCad schematic)
At the start: 9 parts, among them J1 DE15_Socket_HighDensity_Mount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, J2 Conn_01x03_Socket, J3 Conn_01x02_Socket, J4 Conn_01x04_Socket

Commit message: Corrected R2 Link
Parts:
- R2: value 1k -> 10k
Changed lines of the file:
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@@
 			)
 		)
-		(property "Value" "1k"
+		(property "Value" "10k"
 			(at 112.522 72.136 0)
 			(effects
@@
 			)
 		)
-		(property "Datasheet" "https://jlcpcb.com/partdetail/21904-0603WAF1001T5E/C21190"
+		(property "Datasheet" "https://jlcpcb.com/partdetail/16079-0603WAJ0103T5E/C15401"
 			(at 115.57 71.12 0)
 			(effects
